File: hardware/v1-PSMX/v1-PSMX.kicad_pcb (KiCad board)
At the start: 2 copper layers, 91.4 x 48.8 mm, 36 parts, among them IC1 MAX98357AETE+T (L), IC2 MAX98357AETE+T (R), J1 +5v_POWER, J2 Conn_01x04, J3 10118192-0002LF, J4 Serial_Breakout, U1 ESP32-S3-WROOM-1, U2 AZ1084-3.3

Commit message: Added some more labels
Other:
- board text added: "+5V"
- board text added: "GND"
- board text added: "L+"
- board text added: "L-"
- board text added: "R+"
- board text added: "R-"
- board text added: "RX"
- board text added: "TX"
Changed lines of the file:
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@@
   (gr_line (start 187.452 80.264) (end 165.735 80.264) (layer "Edge.Cuts") (width 0.1))
   (gr_circle (center 180.848 104.648) (end 180.848 119.888) (layer "F.CrtYd") (width 0.05) (fill none))
+  (gr_text "+5V" (at 143.764 82.804) (layer "F.SilkS")
+    (effects (font (size 0.381 0.381) (thickness 0.09525)))
+  )
   (gr_text "ESD" (at 151.13 90.424 90) (layer "F.SilkS")
     (effects (font (size 0.381 0.381) (thickness 0.09525)))
@@
     (effects (font (size 0.381 0.381) (thickness 0.09525)))
   )
+  (gr_text "L-" (at 130.81 87.757) (layer "F.SilkS")
+    (effects (font (size 0.381 0.381) (thickness 0.09525)))
+  )
   (gr_text "220kohm" (at 124.968 96.012 90) (layer "F.SilkS")
+    (effects (font (size 0.381 0.381) (thickness 0.09525)))
+  )
+  (gr_text "L+" (at 128.27 87.757) (layer "F.SilkS")
     (effects (font (size 0.381 0.381) (thickness 0.09525)))
   )
@@
     (effects (font (size 0.381 0.381) (thickness 0.09525)))
   )
+  (gr_text "RX" (at 137.287 82.804) (layer "F.SilkS")
+    (effects (font (size 0.381 0.381) (thickness 0.09525)))
+  )
   (gr_text "10uF" (at 131.699 95.885) (layer "F.SilkS")
+    (effects (font (size 0.381 0.381) (thickness 0.09525)))
+  )
+  (gr_text "R+" (at 123.317 87.757) (layer "F.SilkS")
     (effects (font (size 0.381 0.381) (thickness 0.09525)))
   )
@@
     (effects (font (size 0.381 0.381) (thickness 0.09525)))
   )
+  (gr_text "TX" (at 137.287 85.344) (layer "F.SilkS")
+    (effects (font (size 0.381 0.381) (thickness 0.09525)))
+  )
   (gr_text "0.1uF" (at 153.416 107.823) (layer "F.SilkS")
     (effects (font (size 0.381 0.381) (thickness 0.09525)))
@@
   (gr_text "v1-PSMX.test-1" (at 180.975 127.889) (layer "F.SilkS")
     (effects (font (size 1 1) (thickness 0.15)))
+  )
+  (gr_text "GND" (at 143.764 85.344) (layer "F.SilkS")
+    (effects (font (size 0.381 0.381) (thickness 0.09525)))
   )
   (gr_text "10uF" (at 153.416 101.727) (layer "F.SilkS")
@@
     (effects (font (size 0.381 0.381) (thickness 0.09525)))
   )
+  (gr_text "R-" (at 125.73 87.757) (layer "F.SilkS")
+    (effects (font (size 0.381 0.381) (thickness 0.09525)))
+  )

Commit message: msic
Parts:
- moved C11 3.04 mm to (154.9, 101.0)
- moved C10 2.54 mm to (154.9, 98.6)
- moved C12 1.65 mm to (154.9, 107.3)
- moved C13 1.53 mm to (154.9, 109.9)
Routing:
- net +5V: track 114.2 -> 108.6 mm
- net +3.3V: track 110.2 -> 109.5 mm
